File: docs/caliper.kicad_sch (KiCad schematic)
At the start: 8 parts

Commit message: fix transistors from BCE to EBC pinout in schematic
Parts:
- Q? (x2): value Q_NPN_BCE -> Q_NPN_EBC; symbol Device:Q_NPN_BCE -> Device:Q_NPN_EBC
Connections:
- net GND: now also Q?.1 (E), Q?.1 (E); no longer Q?.3 (E), Q?.3 (E)
- net ~{CLK} Out: now also Q?.3 (C); no longer Q?.2 (C)
- net ~{DAT} Out: now also Q?.3 (C); no longer Q?.2 (C)
- net at R?.2: now also Q?.2 (B); no longer Q?.1 (B) (x2)
Changed lines of the file:
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@@
     (pin "1")
   )
-  (symbol (lib_id "Device:Q_NPN_BCE") (at 191.77 121.92 0) (unit 1)
+  (symbol (lib_id "Device:Q_NPN_EBC") (at 191.77 121.92 0) (unit 1)
     (in_bom yes) (on_board yes) (fields_autoplaced)
     (property "Reference" "Q?" (id 0) (at 196.6214 121.0853 0)
       (effects (font (size 1.27 1.27)) (justify left) hide)
     )
-    (property "Value" "Q_NPN_BCE" (id 1) (at 196.6214 123.6222 0)
+    (property "Value" "Q_NPN_EBC" (id 1) (at 196.85 123.19 0)
       (effects (font (size 1.27 1.27)) (justify left) hide)
     )
@@
     (pin "1")
   )
-  (symbol (lib_id "Device:Q_NPN_BCE") (at 181.61 114.3 0) (unit 1)
+  (symbol (lib_id "Device:Q_NPN_EBC") (at 181.61 114.3 0) (unit 1)
     (in_bom yes) (on_board yes) (fields_autoplaced)
     (property "Reference" "Q?" (id 0) (at 186.4614 113.4653 0)
       (effects (font (size 1.27 1.27)) (justify left) hide)
     )
-    (property "Value" "Q_NPN_BCE" (id 1) (at 186.4614 116.0022 0)
+    (property "Value" "Q_NPN_EBC" (id 1) (at 186.69 115.57 0)
       (effects (font (size 1.27 1.27)) (justify left) hide)
     )
@@
     )
     (path "/4a7f1edb-4587-47ea-97db-4c8bebe01214"
-      (reference "Q?") (unit 1) (value "Q_NPN_BCE") (footprint "")
+      (reference "Q?") (unit 1) (value "Q_NPN_EBC") (footprint "")
     )
     (path "/c3fc18e4-72ab-4453-82d7-9983960b0e19"
-      (reference "Q?") (unit 1) (value "Q_NPN_BCE") (footprint "")
+      (reference "Q?") (unit 1) (value "Q_NPN_EBC") (footprint "")
     )
     (path "/0dea59e4-0947-4b42-9006-e9933443abc1"
